Commit message: Salamanca urdf - Display model in RViz with cylinders for wheels; inertia, dimensions, and position settings pending.

File: models/src/salamanca/urdf/mobile_base.urdf.xacro (robot description, xacro)
@@ -47,15 +47,14 @@
     <xacro:property name="battery_height" value="0.1" />
     <xacro:property name="battery_mass" value="1" />
-    <link name="base_footprint" />
-    <link name="base_osb">
-        <visual>
-            <geometry>
-                <mesh filename="package://salamanca/stl/OSB 18mm v28.stl" scale="1 1 1" />
-            </geometry>
-            <origin xyz="0 0 0" rpy="0 0 0" />
-        </visual>
-        <collision>
-            <geometry>
-                <mesh filename="package://salamanca/stl/OSB 18mm v28.stl" scale="1 1 1" />
+    <link name="base_link">
+        <visual>
+            <geometry>
+                <mesh filename="package://salamanca/stl/OSB_18mm_v28.stl" scale="1 1 1" />
+            </geometry>
+            <origin xyz="0 0 0" rpy="0 0 0" />
+        </visual>
+        <collision>
+            <geometry>
+                <mesh filename="package://salamanca/stl/OSB_18mm_v28.stl" scale="1 1 1" />
             </geometry>
             <origin xyz="0 0 0" rpy="0 0 0" />
@@ -64,14 +63,15 @@
             xyz="0 0 0" rpy="0 0 0" />
     </link>
+    <link name="base_footprint"></link>
     <link name="castor_wheel">
         <visual>
             <geometry>
-                <mesh filename="package://salamanca/stl/Castor Wheel 50X19 v4.stl" scale="1 1 1" />
-            </geometry>
-            <origin xyz="0 0 0" rpy="0 0 0" />
-        </visual>
-        <collision>
-            <geometry>
-                <mesh filename="package://salamanca/stl/Castor Wheel 50X19 v4.stl" scale="1 1 1" />
+                <mesh filename="package://salamanca/stl/Castor_Wheel_50X19_v4.stl" scale="1 1 1" />
+            </geometry>
+            <origin xyz="0 0 0" rpy="0 0 0" />
+        </visual>
+        <collision>
+            <geometry>
+                <mesh filename="package://salamanca/stl/Castor_Wheel_50X19_v4.stl" scale="1 1 1" />
             </geometry>
             <origin xyz="0 0 0" rpy="0 0 0" />
@@ -83,5 +83,5 @@
         <visual>
             <geometry>
-                <mesh filename="package://salamanca/stl/Intel_RealSense_Depth_Camera_D435 v3.stl"
+                <mesh filename="package://salamanca/stl/Intel_RealSense_Depth_Camera_D435_v3.stl"
                     scale="1 1 1" />
             </geometry>
@@ -90,5 +90,5 @@
         <collision>
             <geometry>
-                <mesh filename="package://salamanca/stl/Intel_RealSense_Depth_Camera_D435 v3.stl"
+                <mesh filename="package://salamanca/stl/Intel_RealSense_Depth_Camera_D435_v3.stl"
                     scale="1 1 1" />
             </geometry>
@@ -101,11 +101,11 @@
         <visual>
             <geometry>
-                <mesh filename="package://salamanca/stl/Jetson nano v2 v2.stl" scale="1 1 1" />
-            </geometry>
-            <origin xyz="0 0 0" rpy="0 0 0" />
-        </visual>
-        <collision>
-            <geometry>
-                <mesh filename="package://salamanca/stl/Jetson nano v2 v2.stl" scale="1 1 1" />
+                <mesh filename="package://salamanca/stl/Jetson_nano_v2_v2.stl" scale="1 1 1" />
+            </geometry>
+            <origin xyz="0 0 0" rpy="0 0 0" />
+        </visual>
+        <collision>
+            <geometry>
+                <mesh filename="package://salamanca/stl/Jetson_nano_v2_v2.stl" scale="1 1 1" />
             </geometry>
             <origin xyz="0 0 0" rpy="0 0 0" />
@@ -117,11 +117,11 @@
         <visual>
             <geometry>
-                <mesh filename="package://salamanca/stl/ODrive Bothwheel v4.stl" scale="1 1 1" />
-            </geometry>
-            <origin xyz="0 0 0" rpy="0 0 0" />
-        </visual>
-        <collision>
-            <geometry>
-                <mesh filename="package://salamanca/stl/ODrive Bothwheel v4.stl" scale="1 1 1" />
+                <cylinder radius="${odrive_radius}" length="${odrive_height}" />
+            </geometry>
+            <origin xyz="0 0 0" rpy="0 0 0" />
+        </visual>
+        <collision>
+            <geometry>
+                <cylinder radius="${odrive_radius}" length="${odrive_height}" />
             </geometry>
             <origin xyz="0 0 0" rpy="0 0 0" />
@@ -133,11 +133,11 @@
         <visual>
             <geometry>
-                <mesh filename="package://salamanca/stl/rplidar-a2m4-r1 v3.stl" scale="1 1 1" />
-            </geometry>
-            <origin xyz="0 0 0" rpy="0 0 0" />
-        </visual>
-        <collision>
-            <geometry>
-                <mesh filename="package://salamanca/stl/rplidar-a2m4-r1 v3.stl" scale="1 1 1" />
+                <mesh filename="package://salamanca/stl/rplidar_a2m4_r1_v3.stl" scale="1 1 1" />
+            </geometry>
+            <origin xyz="0 0 0" rpy="0 0 0" />
+        </visual>
+        <collision>
+            <geometry>
+                <mesh filename="package://salamanca/stl/rplidar_a2m4_r1_v3.stl" scale="1 1 1" />
             </geometry>
             <origin xyz="0 0 0" rpy="0 0 0" />
@@ -149,11 +149,11 @@
         <visual>
             <geometry>
-                <mesh filename="package://salamanca/stl/Tattu 6S 22.2V 10000Ah v4.stl" scale="1 1 1" />
-            </geometry>
-            <origin xyz="0 0 0" rpy="0 0 0" />
-        </visual>
-        <collision>
-            <geometry>
-                <mesh filename="package://salamanca/stl/Tattu 6S 22.2V 10000Ah v4.stl" scale="1 1 1" />
+                <mesh filename="package://salamanca/stl/Tattu_6S_22_2V_10000Ah_v4.stl" scale="1 1 1" />
+            </geometry>
+            <origin xyz="0 0 0" rpy="0 0 0" />
+        </visual>
+        <collision>
+            <geometry>
+                <mesh filename="package://salamanca/stl/Tattu_6S_22_2V_10000Ah_v4.stl" scale="1 1 1" />
             </geometry>
             <origin xyz="0 0 0" rpy="0 0 0" />
@@ -162,3 +162,53 @@
             xyz="0 0 0" rpy="0 0 0" />
     </link>
+    <joint name="castor_joint" type="fixed">
+        <parent link="base_link" />
+        <child link="castor_wheel" />
+        <origin xyz="0 0 -0.15" rpy="0 0 0" /> <!-- Adjust xyz to position battery relative to base_link -->
+    </joint>
+    <joint name="base_joint" type="fixed">
+        <parent link="base_link" />
+        <child link="base_footprint" />
+        <origin xyz="0 0 -0.10" rpy="0 0 0" /> <!-- Adjust xyz to position battery relative to base_link -->
+    </joint>
+    <!-- Battery Joint -->
+    <joint name="battery_joint" type="fixed">
+        <parent link="base_link" />
+        <child link="tattu_battery" />
+        <origin xyz="0 0 -0.05" rpy="0 0 0" /> <!-- Adjust xyz to position battery relative to base_link -->
+    </joint>
+    <!-- RealSense Camera Joint -->
+    <joint name="realsense_joint" type="fixed">
+        <parent link="base_link" />
+        <child link="realsense_camera" />
+        <origin xyz="0.05 0 0.1" rpy="0 0 0" /> <!-- Adjust xyz to position RealSense relative to base_link -->
+    </joint>
+    <!-- RPLIDAR Mount Joint -->
+    <joint name="rplidar_mount_joint" type="fixed">
+        <parent link="base_link" />
+        <child link="rplidar_a2_mount" />
+        <origin xyz="0 0 0.15" rpy="0 0 0" /> <!-- Adjust xyz to position RPLIDAR relative to base_link -->
+    </joint>
+    <!-- Jetson Nano Joint -->
+    <joint name="jetson_joint" type="fixed">
+        <parent link="base_link" />
+        <child link="jetson_nano" />
+        <origin xyz="0 0.05 0.05" rpy="0 0 0" /> <!-- Adjust xyz to position Jetson Nano relative to base_link -->
+    </joint>
+    <!-- Left Wheel Joint -->
+    <joint name="left_wheel_joint" type="revolute">
+        <parent link="base_link" />
+        <child link="odrive_bothwheel" />
+        <origin xyz="0 -0.1 0" rpy="0 0 0" /> <!-- Adjust xyz to position left wheel relative to base_link -->
+        <axis xyz="0 1 0" />
+        <limit lower="-1.5708" upper="1.5708" effort="1" velocity="10" />
+    </joint>
+    <!-- Right Wheel Joint -->
+    <joint name="right_wheel_joint" type="revolute">
+        <parent link="base_link" />
+        <child link="odrive_bothwheel" />
+        <origin xyz="0 0.1 0" rpy="0 0 0" /> <!-- Adjust xyz to position right wheel relative to base_link -->
+        <axis xyz="0 1 0" />
+        <limit lower="-1.5708" upper="1.5708" effort="1" velocity="10" />
+    </joint>
 </robot>

Commit message: Salamanca urdf - Display model in RViz with cylinders for wheels; position settings pending.

File: models/src/salamanca/urdf/mobile_base.urdf.xacro (robot description, xacro)
@@ -1,60 +1,61 @@
 <?xml version="1.0"?>
 <robot xmlns:xacro="http://www.ros.org/wiki/xacro">
+    <xacro:property name="scale_factor" value="0.001" />
     <!--Base size
     (TODO: set teh correct dimensions)-->
-    <xacro:property name="base_length" value="0.1" />
-    <xacro:property name="base_width" value="0.1" />
-    <xacro:property name="base_height" value="0.1" />
+    <xacro:property name="base_length" value="0.43" />
+    <xacro:property name="base_width" value="0.245" />
+    <xacro:property name="base_height" value="0.018" />
     <xacro:property name="base_mass" value="1" />
     <!--Castor wheel size
     (TODO: set teh correct dimensions)-->
-    <xacro:property name="castor_radius" value="0.1" />
-    <xacro:property name="castor_height" value="0.1" />
+    <xacro:property name="castor_radius" value="0.022" />
+    <xacro:property name="castor_height" value="0.007" />
     <xacro:property name="castor_mass" value="1" />
     <!--Realsense size
     (TODO: set teh correct dimensions)-->
-    <xacro:property name="realsense_length" value="0.1" />
-    <xacro:property name="realsense_width" value="0.1" />
-    <xacro:property name="realsense_height" value="0.1" />
+    <xacro:property name="realsense_length" value="0.09" />
+    <xacro:property name="realsense_width" value="0.025" />
+    <xacro:property name="realsense_height" value="0.025" />
     <xacro:property name="realsense_mass" value="1" />
     <!--Jetson size
     (TODO: set teh correct dimensions)-->
-    <xacro:property name="jetson_length" value="0.1" />
-    <xacro:property name="jetson_width" value="0.1" />
-    <xacro:property name="jetson_height" value="0.1" />
+    <xacro:property name="jetson_length" value="0.10" />
+    <xacro:property name="jetson_width" value="0.079" />
+    <xacro:property name="jetson_height" value="0.029" />
     <xacro:property name="jetson_mass" value="1" />
     <!--Odrive size
     (TODO: set teh correct dimensions)-->
-    <xacro:property name="odrive_radius" value="0.1" />
-    <xacro:property name="odrive_height" value="0.1" />
+    <xacro:property name="odrive_radius" value="0.0855" />
+    <xacro:property name="odrive_height" value="0.045" />
     <xacro:property name="odrive_mass" value="1" />
     <!--Realsense adapter size
     (TODO: set teh correct dimensions)-->
-    <xacro:property name="realsense_adapter_length" value="0.1" />
-    <xacro:property name="realsense_adapter_width" value="0.1" />
-    <xacro:property name="realsense_adapter_height" value="0.1" />
+    <xacro:property name="realsense_adapter_length" value="0.09" />
+    <xacro:property name="realsense_adapter_width" value="0.025" />
+    <xacro:property name="realsense_adapter_height" value="0.025" />
     <xacro:property name="realsense_adapter_mass" value="1" />
     <!--Rplidar mount size
     (TODO: set teh correct dimensions)-->
-    <xacro:property name="rplidar_mount_length" value="0.1" />
-    <xacro:property name="rplidar_mount_width" value="0.1" />
-    <xacro:property name="rplidar_mount_height" value="0.1" />
+    <xacro:property name="rplidar_mount_length" value="0.075" />
+    <xacro:property name="rplidar_mount_width" value="0.075" />
+    <xacro:property name="rplidar_mount_height" value="0.045" />
     <xacro:property name="rplidar_mount_mass" value="1" />
     <!--Tattu battery size
     (TODO: set teh correct dimensions)-->
-    <xacro:property name="battery_length" value="0.1" />
-    <xacro:property name="battery_width" value="0.1" />
-    <xacro:property name="battery_height" value="0.1" />
+    <xacro:property name="battery_length" value="0.17" />
+    <xacro:property name="battery_width" value="0.058" />
+    <xacro:property name="battery_height" value="0.062" />
     <xacro:property name="battery_mass" value="1" />
     <link name="base_link">
         <visual>
             <geometry>
-                <mesh filename="package://salamanca/stl/OSB_18mm_v28.stl" scale="1 1 1" />
-            </geometry>
-            <origin xyz="0 0 0" rpy="0 0 0" />
-        </visual>
-        <collision>
-            <geometry>
-                <mesh filename="package://salamanca/stl/OSB_18mm_v28.stl" scale="1 1 1" />
+                <mesh filename="package://salamanca/stl/OSB_18mm_v28.stl" scale="${scale_factor} ${scale_factor} ${scale_factor}" />
+            </geometry>
+            <origin xyz="0 0 0" rpy="0 0 0" />
+        </visual>
+        <collision>
+            <geometry>
+                <mesh filename="package://salamanca/stl/OSB_18mm_v28.stl" scale="${scale_factor} ${scale_factor} ${scale_factor}" />
             </geometry>
             <origin xyz="0 0 0" rpy="0 0 0" />
@@ -67,11 +68,11 @@
         <visual>
             <geometry>
-                <mesh filename="package://salamanca/stl/Castor_Wheel_50X19_v4.stl" scale="1 1 1" />
-            </geometry>
-            <origin xyz="0 0 0" rpy="0 0 0" />
-        </visual>
-        <collision>
-            <geometry>
-                <mesh filename="package://salamanca/stl/Castor_Wheel_50X19_v4.stl" scale="1 1 1" />
+                <mesh filename="package://salamanca/stl/Castor_Wheel_50X19_v4.stl" scale="${scale_factor} ${scale_factor} ${scale_factor}" />
+            </geometry>
+            <origin xyz="0 0 0" rpy="0 0 0" />
+        </visual>
+        <collision>
+            <geometry>
+                <mesh filename="package://salamanca/stl/Castor_Wheel_50X19_v4.stl" scale="${scale_factor} ${scale_factor} ${scale_factor}" />
             </geometry>
             <origin xyz="0 0 0" rpy="0 0 0" />
@@ -84,5 +85,5 @@
             <geometry>
                 <mesh filename="package://salamanca/stl/Intel_RealSense_Depth_Camera_D435_v3.stl"
-                    scale="1 1 1" />
+                scale="${scale_factor} ${scale_factor} ${scale_factor}" />
             </geometry>
             <origin xyz="0 0 0" rpy="0 0 0" />
@@ -91,5 +92,5 @@
             <geometry>
                 <mesh filename="package://salamanca/stl/Intel_RealSense_Depth_Camera_D435_v3.stl"
-                    scale="1 1 1" />
+                scale="${scale_factor} ${scale_factor} ${scale_factor}" />
             </geometry>
             <origin xyz="0 0 0" rpy="0 0 0" />
@@ -101,11 +102,11 @@
         <visual>
             <geometry>
-                <mesh filename="package://salamanca/stl/Jetson_nano_v2_v2.stl" scale="1 1 1" />
-            </geometry>
-            <origin xyz="0 0 0" rpy="0 0 0" />
-        </visual>
-        <collision>
-            <geometry>
-                <mesh filename="package://salamanca/stl/Jetson_nano_v2_v2.stl" scale="1 1 1" />
+                <mesh filename="package://salamanca/stl/Jetson_nano_v2_v2.stl" scale="${scale_factor} ${scale_factor} ${scale_factor}" />
+            </geometry>
+            <origin xyz="0 0 0" rpy="0 0 0" />
+        </visual>
+        <collision>
+            <geometry>
+                <mesh filename="package://salamanca/stl/Jetson_nano_v2_v2.stl" scale="${scale_factor} ${scale_factor} ${scale_factor}" />
             </geometry>
             <origin xyz="0 0 0" rpy="0 0 0" />
@@ -119,5 +120,5 @@
                 <cylinder radius="${odrive_radius}" length="${odrive_height}" />
             </geometry>
-            <origin xyz="0 0 0" rpy="0 0 0" />
+            <origin xyz="0 0 0" rpy="1.5708 0 0" />
         </visual>
         <collision>
@@ -125,5 +126,5 @@
                 <cylinder radius="${odrive_radius}" length="${odrive_height}" />
             </geometry>
-            <origin xyz="0 0 0" rpy="0 0 0" />
+            <origin xyz="0 0 0" rpy="1.5708 0 0" />
         </collision>
         <xacro:cylinder_inertia m="${odrive_mass}" r="${odrive_radius}" h="${odrive_height}"
@@ -133,13 +134,13 @@
         <visual>
             <geometry>
-                <mesh filename="package://salamanca/stl/rplidar_a2m4_r1_v3.stl" scale="1 1 1" />
-            </geometry>
-            <origin xyz="0 0 0" rpy="0 0 0" />
-        </visual>
-        <collision>
-            <geometry>
-                <mesh filename="package://salamanca/stl/rplidar_a2m4_r1_v3.stl" scale="1 1 1" />
-            </geometry>
-            <origin xyz="0 0 0" rpy="0 0 0" />
+                <mesh filename="package://salamanca/stl/rplidar_a2m4_r1_v3.stl" scale="${scale_factor} ${scale_factor} ${scale_factor}" />
+            </geometry>
+            <origin xyz="0 0 0" rpy="0 1.5708 0" />
+        </visual>
+        <collision>
+            <geometry>
+                <mesh filename="package://salamanca/stl/rplidar_a2m4_r1_v3.stl" scale="${scale_factor} ${scale_factor} ${scale_factor}" />
+            </geometry>
+            <origin xyz="0 0 0" rpy="0 1.5708 0" />
         </collision>
         <xacro:box_inertia m="${rplidar_mount_mass}" l="${rplidar_mount_length}" w="${rplidar_mount_width}" h="${rplidar_mount_height}"
@@ -149,11 +150,11 @@
         <visual>
             <geometry>
-                <mesh filename="package://salamanca/stl/Tattu_6S_22_2V_10000Ah_v4.stl" scale="1 1 1" />
-            </geometry>
-            <origin xyz="0 0 0" rpy="0 0 0" />
-        </visual>
-        <collision>
-            <geometry>
-                <mesh filename="package://salamanca/stl/Tattu_6S_22_2V_10000Ah_v4.stl" scale="1 1 1" />
+                <mesh filename="package://salamanca/stl/Tattu_6S_22_2V_10000Ah_v4.stl" scale="${scale_factor} ${scale_factor} ${scale_factor}" />
+            </geometry>
+            <origin xyz="0 0 0" rpy="0 0 0" />
+        </visual>
+        <collision>
+            <geometry>
+                <mesh filename="package://salamanca/stl/Tattu_6S_22_2V_10000Ah_v4.stl" scale="${scale_factor} ${scale_factor} ${scale_factor}" />
             </geometry>
             <origin xyz="0 0 0" rpy="0 0 0" />
@@ -162,9 +163,4 @@
             xyz="0 0 0" rpy="0 0 0" />
     </link>
-    <joint name="castor_joint" type="fixed">
-        <parent link="base_link" />
-        <child link="castor_wheel" />
-        <origin xyz="0 0 -0.15" rpy="0 0 0" /> <!-- Adjust xyz to position battery relative to base_link -->
-    </joint>
     <joint name="base_joint" type="fixed">
         <parent link="base_link" />
@@ -172,41 +168,47 @@
         <origin xyz="0 0 -0.10" rpy="0 0 0" /> <!-- Adjust xyz to position battery relative to base_link -->
     </joint>
-    <!-- Battery Joint -->
+    <!-- Joint Castor Wheel - Przód pod podstawą -->
+    <joint name="castor_joint" type="fixed">
+        <parent link="base_link" />
+        <child link="castor_wheel" />
+        <origin xyz="0 0 0" rpy="0 0 0" />
+    </joint>
+    <!-- Joint RPLIDAR - Środek podstawy -->
+    <joint name="rplidar_mount_joint" type="fixed">
+        <parent link="base_link" />
+        <child link="rplidar_a2_mount" />
+        <origin xyz="0 0 0" rpy="0 0 0" />
+    </joint>
+    <!-- Joint RealSense - Przód nad lidar -->
+    <joint name="realsense_joint" type="fixed">
+        <parent link="base_link" />
+        <child link="realsense_camera" />
+        <origin xyz="0 0 0" rpy="0 0 0" />
+    </joint>
+    <!-- Joint Tattu Battery - Przód za RealSense -->
     <joint name="battery_joint" type="fixed">
         <parent link="base_link" />
         <child link="tattu_battery" />
-        <origin xyz="0 0 -0.05" rpy="0 0 0" /> <!-- Adjust xyz to position battery relative to base_link -->
-    </joint>
-    <!-- RealSense Camera Joint -->
-    <joint name="realsense_joint" type="fixed">
-        <parent link="base_link" />
-        <child link="realsense_camera" />
-        <origin xyz="0.05 0 0.1" rpy="0 0 0" /> <!-- Adjust xyz to position RealSense relative to base_link -->
-    </joint>
-    <!-- RPLIDAR Mount Joint -->
-    <joint name="rplidar_mount_joint" type="fixed">
-        <parent link="base_link" />
-        <child link="rplidar_a2_mount" />
-        <origin xyz="0 0 0.15" rpy="0 0 0" /> <!-- Adjust xyz to position RPLIDAR relative to base_link -->
-    </joint>
-    <!-- Jetson Nano Joint -->
+        <origin xyz="0 0 0" rpy="0 0 0" />
+    </joint>
+    <!-- Joint Jetson Nano - Tylna część podstawy -->
     <joint name="jetson_joint" type="fixed">
         <parent link="base_link" />
         <child link="jetson_nano" />
-        <origin xyz="0 0.05 0.05" rpy="0 0 0" /> <!-- Adjust xyz to position Jetson Nano relative to base_link -->
-    </joint>
-    <!-- Left Wheel Joint -->
+        <origin xyz="0 0 0" rpy="0 0 0" />
+    </joint>
+    <!-- Joint Left Wheel - Tylna lewa strona podstawy -->
     <joint name="left_wheel_joint" type="revolute">
         <parent link="base_link" />
         <child link="odrive_bothwheel" />
-        <origin xyz="0 -0.1 0" rpy="0 0 0" /> <!-- Adjust xyz to position left wheel relative to base_link -->
+        <origin xyz="${-base_length / 2 - 0.1} ${-base_width / 2} ${odrive_radius}" rpy="0 0 0" />
         <axis xyz="0 1 0" />
         <limit lower="-1.5708" upper="1.5708" effort="1" velocity="10" />
     </joint>
-    <!-- Right Wheel Joint -->
+    <!-- Joint Right Wheel - Tylna prawa strona podstawy -->
     <joint name="right_wheel_joint" type="revolute">
         <parent link="base_link" />
         <child link="odrive_bothwheel" />
-        <origin xyz="0 0.1 0" rpy="0 0 0" /> <!-- Adjust xyz to position right wheel relative to base_link -->
+        <origin xyz="${-base_length / 2 + 0.1} ${base_width / 2} ${odrive_radius}" rpy="0 0 0" />
         <axis xyz="0 1 0" />
         <limit lower="-1.5708" upper="1.5708" effort="1" velocity="10" />
