Commit message: Realsense ROS2 node - beginning

File: models/install/salamanca/share/salamanca/urdf/mobile_base.urdf.xacro (robot description, xacro)
@@ -1,62 +1,51 @@
 <?xml version="1.0"?>
 <robot xmlns:xacro="http://www.ros.org/wiki/xacro">
-    <!--Base size
-    (TODO: set teh correct dimensions)-->
-    <xacro:property name="base_length" value="0.1" />
-    <xacro:property name="base_width" value="0.1" />
-    <xacro:property name="base_height" value="0.1" />
+    <xacro:property name="scale_factor" value="0.001" />
+    <!--Base size -->
+    <xacro:property name="base_length" value="0.43" />
+    <xacro:property name="base_width" value="0.245" />
+    <xacro:property name="base_height" value="0.018" />
     <xacro:property name="base_mass" value="1" />
-    <!--Castor wheel size
-    (TODO: set teh correct dimensions)-->
-    <xacro:property name="castor_radius" value="0.1" />
-    <xacro:property name="castor_height" value="0.1" />
-    <xacro:property name="castor_mass" value="1" />
-    <!--Realsense size
-    (TODO: set teh correct dimensions)-->
-    <xacro:property name="realsense_length" value="0.1" />
-    <xacro:property name="realsense_width" value="0.1" />
-    <xacro:property name="realsense_height" value="0.1" />
-    <xacro:property name="realsense_mass" value="1" />
-    <!--Jetson size
-    (TODO: set teh correct dimensions)-->
-    <xacro:property name="jetson_length" value="0.1" />
-    <xacro:property name="jetson_width" value="0.1" />
-    <xacro:property name="jetson_height" value="0.1" />
-    <xacro:property name="jetson_mass" value="1" />
+    <!--Castor wheel size -->
+    <xacro:property name="castor_radius" value="0.022" />
+    <xacro:property name="castor_height" value="0.007" />
+    <xacro:property name="castor_mass" value="0.08" />
+    <!--Realsense size -->
+    <xacro:property name="realsense_length" value="0.09" />
+    <xacro:property name="realsense_width" value="0.025" />
+    <xacro:property name="realsense_height" value="0.025" />
+    <xacro:property name="realsense_mass" value="0.072" />
+    <!--Jetson size -->
+    <xacro:property name="jetson_length" value="0.10" />
+    <xacro:property name="jetson_width" value="0.079" />
+    <xacro:property name="jetson_height" value="0.029" />
+    <xacro:property name="jetson_mass" value="0.28" />
     <!--Odrive size
     (TODO: set teh correct dimensions)-->
-    <xacro:property name="odrive_radius" value="0.1" />
-    <xacro:property name="odrive_height" value="0.1" />
-    <xacro:property name="odrive_mass" value="1" />
-    <!--Realsense adapter size
-    (TODO: set teh correct dimensions)-->
-    <xacro:property name="realsense_adapter_length" value="0.1" />
-    <xacro:property name="realsense_adapter_width" value="0.1" />
-    <xacro:property name="realsense_adapter_height" value="0.1" />
-    <xacro:property name="realsense_adapter_mass" value="1" />
-    <!--Rplidar mount size
-    (TODO: set teh correct dimensions)-->
-    <xacro:property name="rplidar_mount_length" value="0.1" />
-    <xacro:property name="rplidar_mount_width" value="0.1" />
-    <xacro:property name="rplidar_mount_height" value="0.1" />
-    <xacro:property name="rplidar_mount_mass" value="1" />
-    <!--Tattu battery size
-    (TODO: set teh correct dimensions)-->
-    <xacro:property name="battery_length" value="0.1" />
-    <xacro:property name="battery_width" value="0.1" />
-    <xacro:property name="battery_height" value="0.1" />
-    <xacro:property name="battery_mass" value="1" />
+    <xacro:property name="odrive_radius" value="0.0855" />
+    <xacro:property name="odrive_height" value="0.045" />
+    <xacro:property name="odrive_mass" value="2.2" />
+    <!--Rplidar mount size-->
+    <xacro:property name="rplidar_mount_length" value="0.075" />
+    <xacro:property name="rplidar_mount_width" value="0.075" />
+    <xacro:property name="rplidar_mount_height" value="0.045" />
+    <xacro:property name="rplidar_mount_mass" value="0.34" />
+    <!--Tattu battery size -->
+    <xacro:property name="battery_length" value="0.17" />
+    <xacro:property name="battery_width" value="0.058" />
+    <xacro:property name="battery_height" value="0.062" />
+    <xacro:property name="battery_mass" value="1.974" />
     <link name="base_link">
         <visual>
             <geometry>
-                <mesh filename="package://salamanca/stl/OSB_18mm_v28.stl" scale="1 1 1" />
-            </geometry>
-            <origin xyz="0 0 0" rpy="0 0 0" />
-        </visual>
-        <collision>
-            <geometry>
-                <mesh filename="package://salamanca/stl/OSB_18mm_v28.stl" scale="1 1 1" />
-            </geometry>
-            <origin xyz="0 0 0" rpy="0 0 0" />
+                <mesh filename="package://salamanca/stl/base_link.stl" scale="${scale_factor} ${scale_factor} ${scale_factor}" />
+            </geometry>
+            <origin xyz="0 0 0" rpy="0 0 0" />
+        </visual>
+        <collision>
+            <geometry>
+                <mesh filename="package://salamanca/stl/base_link.stl" scale="${scale_factor} ${scale_factor} ${scale_factor}" />
+            </geometry>
+            <origin xyz="${-base_length/2} 0 0" rpy="0 0 0" />
         </collision>
         <xacro:box_inertia m="${base_mass}" l="${base_length}" w="${base_width}" h="${base_height}"
@@ -67,11 +56,11 @@
         <visual>
             <geometry>
-                <mesh filename="package://salamanca/stl/Castor_Wheel_50X19_v4.stl" scale="1 1 1" />
-            </geometry>
-            <origin xyz="0 0 0" rpy="0 0 0" />
-        </visual>
-        <collision>
-            <geometry>
-                <mesh filename="package://salamanca/stl/Castor_Wheel_50X19_v4.stl" scale="1 1 1" />
+                <mesh filename="package://salamanca/stl/castor_wheel.stl" scale="${scale_factor} ${scale_factor} ${scale_factor}" />
+            </geometry>
+            <origin xyz="0 0 0" rpy="0 0 0" />
+        </visual>
+        <collision>
+            <geometry>
+                <mesh filename="package://salamanca/stl/castor_wheel.stl" scale="${scale_factor} ${scale_factor} ${scale_factor}" />
             </geometry>
             <origin xyz="0 0 0" rpy="0 0 0" />
@@ -83,13 +72,13 @@
         <visual>
             <geometry>
-                <mesh filename="package://salamanca/stl/Intel_RealSense_Depth_Camera_D435_v3.stl"
-                    scale="1 1 1" />
-            </geometry>
-            <origin xyz="0 0 0" rpy="0 0 0" />
-        </visual>
-        <collision>
-            <geometry>
-                <mesh filename="package://salamanca/stl/Intel_RealSense_Depth_Camera_D435_v3.stl"
-                    scale="1 1 1" />
+                <mesh filename="package://salamanca/stl/realsense_camera.stl"
+                scale="${scale_factor} ${scale_factor} ${scale_factor}" />
+            </geometry>
+            <origin xyz="0 0 0" rpy="0 0 0" />
+        </visual>
+        <collision>
+            <geometry>
+                <mesh filename="package://salamanca/stl/realsense_camera.stl"
+                scale="${scale_factor} ${scale_factor} ${scale_factor}" />
             </geometry>
             <origin xyz="0 0 0" rpy="0 0 0" />
@@ -101,11 +90,11 @@
         <visual>
             <geometry>
-                <mesh filename="package://salamanca/stl/Jetson_nano_v2_v2.stl" scale="1 1 1" />
-            </geometry>
-            <origin xyz="0 0 0" rpy="0 0 0" />
-        </visual>
-        <collision>
-            <geometry>
-                <mesh filename="package://salamanca/stl/Jetson_nano_v2_v2.stl" scale="1 1 1" />
+                <mesh filename="package://salamanca/stl/jetson_nano.stl" scale="${scale_factor} ${scale_factor} ${scale_factor}" />
+            </geometry>
+            <origin xyz="0 0 0" rpy="0 0 0" />
+        </visual>
+        <collision>
+            <geometry>
+                <mesh filename="package://salamanca/stl/jetson_nano.stl" scale="${scale_factor} ${scale_factor} ${scale_factor}" />
             </geometry>
             <origin xyz="0 0 0" rpy="0 0 0" />
@@ -114,30 +103,46 @@
             xyz="0 0 0" rpy="0 0 0" />
     </link>
-    <link name="odrive_bothwheel">
-        <visual>
-            <geometry>
-                <cylinder radius="${odrive_radius}" length="${odrive_height}" />
-            </geometry>
-            <origin xyz="0 0 0" rpy="0 0 0" />
-        </visual>
-        <collision>
-            <geometry>
-                <cylinder radius="${odrive_radius}" length="${odrive_height}" />
-            </geometry>
-            <origin xyz="0 0 0" rpy="0 0 0" />
+    <link name="odrive_bothwheel_r">
+        <visual>
+            <geometry>
+                <cylinder radius="${odrive_radius}" length="${odrive_height}" />
+            </geometry>
+            <origin xyz="0 0 0" rpy="1.5708 0 0" />
+        </visual>
+        <collision>
+            <geometry>
+                <cylinder radius="${odrive_radius}" length="${odrive_height}" />
+            </geometry>
+            <origin xyz="0 0 0" rpy="1.5708 0 0" />
         </collision>
         <xacro:cylinder_inertia m="${odrive_mass}" r="${odrive_radius}" h="${odrive_height}"
             xyz="0 0 0" rpy="0 0 0" />
     </link>
+    <link name="odrive_bothwheel_l">
+        <visual>
+            <geometry>
+                <cylinder radius="${odrive_radius}" length="${odrive_height}" />
+            </geometry>
+            <origin xyz="0 0 0" rpy="1.5708 0 0" />
+        </visual>
+        <collision>
+            <geometry>
+                <cylinder radius="${odrive_radius}" length="${odrive_height}" />
+            </geometry>
+            <origin xyz="0 0 0" rpy="1.5708 0 0" />
+        </collision>
+        <xacro:cylinder_inertia m="${odrive_mass}" r="${odrive_radius}" h="${odrive_height}"
+            xyz="0 0 0" rpy="0 0 0" />
+    </link>
     <link name="rplidar_a2_mount">
         <visual>
             <geometry>
-                <mesh filename="package://salamanca/stl/rplidar_a2m4_r1_v3.stl" scale="1 1 1" />
-            </geometry>
-            <origin xyz="0 0 0" rpy="0 0 0" />
-        </visual>
-        <collision>
-            <geometry>
-                <mesh filename="package://salamanca/stl/rplidar_a2m4_r1_v3.stl" scale="1 1 1" />
+                <mesh filename="package://salamanca/stl/rplidar_a2_mount.stl" scale="${scale_factor} ${scale_factor} ${scale_factor}" />
+            </geometry>
+            <origin xyz="0 0 0" rpy="0 0 0" />
+        </visual>
+        <collision>
+            <geometry>
+                <mesh filename="package://salamanca/stl/rplidar_a2_mount.stl" scale="${scale_factor} ${scale_factor} ${scale_factor}" />
             </geometry>
             <origin xyz="0 0 0" rpy="0 0 0" />
@@ -149,11 +154,11 @@
         <visual>
             <geometry>
-                <mesh filename="package://salamanca/stl/Tattu_6S_22_2V_10000Ah_v4.stl" scale="1 1 1" />
-            </geometry>
-            <origin xyz="0 0 0" rpy="0 0 0" />
-        </visual>
-        <collision>
-            <geometry>
-                <mesh filename="package://salamanca/stl/Tattu_6S_22_2V_10000Ah_v4.stl" scale="1 1 1" />
+                <mesh filename="package://salamanca/stl/tattu_battery.stl" scale="${scale_factor} ${scale_factor} ${scale_factor}" />
+            </geometry>
+            <origin xyz="0 0 0" rpy="0 0 0" />
+        </visual>
+        <collision>
+            <geometry>
+                <mesh filename="package://salamanca/stl/tattu_battery.stl" scale="${scale_factor} ${scale_factor} ${scale_factor}" />
             </geometry>
             <origin xyz="0 0 0" rpy="0 0 0" />
@@ -162,51 +167,45 @@
             xyz="0 0 0" rpy="0 0 0" />
     </link>
+    <joint name="base_joint" type="fixed">
+        <parent link="base_link" />
+        <child link="base_footprint" />
+        <origin xyz="0 0 ${-odrive_radius+base_height}" rpy="0 0 0" />
+    </joint>
     <joint name="castor_joint" type="fixed">
         <parent link="base_link" />
         <child link="castor_wheel" />
-        <origin xyz="0 0 -0.15" rpy="0 0 0" /> <!-- Adjust xyz to position battery relative to base_link -->
-    </joint>
-    <joint name="base_joint" type="fixed">
-        <parent link="base_link" />
-        <child link="base_footprint" />
-        <origin xyz="0 0 -0.10" rpy="0 0 0" /> <!-- Adjust xyz to position battery relative to base_link -->
-    </joint>
-    <!-- Battery Joint -->
+        <origin xyz="${-(2/7)*base_length + 0.01} 0 0" rpy="0 0 0" />
+    </joint>
+    <joint name="rplidar_mount_joint" type="fixed">
+        <parent link="base_link" />
+        <child link="rplidar_a2_mount" />
+        <origin xyz="0 0 0.095" rpy="0 0 0" />
+    </joint>
+    <joint name="realsense_joint" type="fixed">
+        <parent link="base_link" />
+        <child link="realsense_camera" />
+        <origin xyz="${(-base_length/2)+realsense_width} 0 ${base_height}" rpy="0 0 0" />
+    </joint>
     <joint name="battery_joint" type="fixed">
         <parent link="base_link" />
         <child link="tattu_battery" />
-        <origin xyz="0 0 -0.05" rpy="0 0 0" /> <!-- Adjust xyz to position battery relative to base_link -->
-    </joint>
-    <!-- RealSense Camera Joint -->
-    <joint name="realsense_joint" type="fixed">
-        <parent link="base_link" />
-        <child link="realsense_camera" />
-        <origin xyz="0.05 0 0.1" rpy="0 0 0" /> <!-- Adjust xyz to position RealSense relative to base_link -->
-    </joint>
-    <!-- RPLIDAR Mount Joint -->
-    <joint name="rplidar_mount_joint" type="fixed">
-        <parent link="base_link" />
-        <child link="rplidar_a2_mount" />
-        <origin xyz="0 0 0.15" rpy="0 0 0" /> <!-- Adjust xyz to position RPLIDAR relative to base_link -->
-    </joint>
-    <!-- Jetson Nano Joint -->
+        <origin xyz="-0.08 0 ${base_height}" rpy="0 0 0" />
+    </joint>
     <joint name="jetson_joint" type="fixed">
         <parent link="base_link" />
         <child link="jetson_nano" />
-        <origin xyz="0 0.05 0.05" rpy="0 0 0" /> <!-- Adjust xyz to position Jetson Nano relative to base_link -->
-    </joint>
-    <!-- Left Wheel Joint -->
+        <origin xyz="${base_length/3} 0 ${base_height}" rpy="0 0 0" />
+    </joint>
     <joint name="left_wheel_joint" type="revolute">
         <parent link="base_link" />
-        <child link="odrive_bothwheel" />
-        <origin xyz="0 -0.1 0" rpy="0 0 0" /> <!-- Adjust xyz to position left wheel relative to base_link -->
+        <child link="odrive_bothwheel_l" />
+        <origin xyz="${odrive_radius + 0.04} ${(-base_width / 2) - (odrive_height/2)} ${base_height/2}" rpy="0 0 0" />
         <axis xyz="0 1 0" />
         <limit lower="-1.5708" upper="1.5708" effort="1" velocity="10" />
     </joint>
-    <!-- Right Wheel Joint -->
     <joint name="right_wheel_joint" type="revolute">
         <parent link="base_link" />
-        <child link="odrive_bothwheel" />
-        <origin xyz="0 0.1 0" rpy="0 0 0" /> <!-- Adjust xyz to position right wheel relative to base_link -->
+        <child link="odrive_bothwheel_r" />
+        <origin xyz="${odrive_radius + 0.04} ${(base_width / 2) + (odrive_height/2)} ${base_height/2}" rpy="0 0 0" />
         <axis xyz="0 1 0" />
         <limit lower="-1.5708" upper="1.5708" effort="1" velocity="10" />
