Commit message: Work in progress

File: src/pbl_description/urdf/mobile_base.urdf.xacro (robot description, xacro)
@@ -36,4 +36,5 @@
     <xacro:property name="battery_height" value="0.062" />
     <xacro:property name="battery_mass" value="1.974" />
+    <link name="base_footprint"></link>
     <link name="base_link">
         <visual>
@@ -47,10 +48,9 @@
                 <mesh filename="package://pbl_description/stl/base_link.stl" scale="${scale_factor} ${scale_factor} ${scale_factor}" />
             </geometry>
-            <origin xyz="${-base_length/2} 0 0" rpy="0 0 0" />
+            <origin xyz="0 0 0" rpy="0 0 0" />
         </collision>
         <xacro:box_inertia m="${base_mass}" l="${base_length}" w="${base_width}" h="${base_height}"
             xyz="0 0 0" rpy="0 0 0" />
     </link>
-    <link name="base_footprint"></link>
     <link name="castor_wheel">
         <visual>
@@ -202,5 +202,5 @@
         <origin xyz="${odrive_radius + 0.04} ${(-base_width / 2) - (odrive_height/2)} ${base_height/2}" rpy="0 0 0" />
         <axis xyz="0 1 0" />
-        <limit lower="-1.5708" upper="1.5708" effort="1" velocity="10" />
+        <limit lower="-3.14159" upper="3.14159" effort="1" velocity="10" />
     </joint>
     <joint name="right_wheel_joint" type="revolute">
@@ -209,5 +209,5 @@
         <origin xyz="${odrive_radius + 0.04} ${(base_width / 2) + (odrive_height/2)} ${base_height/2}" rpy="0 0 0" />
         <axis xyz="0 1 0" />
-        <limit lower="-1.5708" upper="1.5708" effort="1" velocity="10" />
+        <limit lower="-3.14159" upper="3.14159" effort="1" velocity="10" />
     </joint>
 </robot>

File: src/pbl_description/urdf/mobile_base_gazebo.xacro (robot description, xacro)
@@ -20,6 +20,6 @@
             <update_rate>50</update_rate>
             <!-- wheels -->
-            <left_joint>base_left_wheel_joint</left_joint>
-            <right_joint>base_right_wheel_joint</right_joint>
+            <left_joint>left_wheel_joint</left_joint>
+            <right_joint>right_wheel_joint</right_joint>
             <!-- kinematics -->
             <wheel_separation>0.45</wheel_separation>
@@ -36,3 +36,34 @@
         </plugin>
     </gazebo>
+    <!-- Plugin Gazebo for lidar -->
+    <gazebo reference="rplidar_a2_mount">
+        <sensor type="ray" name="lidar_sensor">
+        <pose>0 0 0 0 0 0</pose>
+        <visualize>true</visualize>
+        <update_rate>10</update_rate>
+        <ray>
+            <scan>
+            <horizontal>
+                <samples>360</samples>
+                <resolution>1</resolution>
+                <min_angle>-3.14159</min_angle>
+                <max_angle>3.14159</max_angle>
+            </horizontal>
+            </scan>
+            <range>
+            <min>0.15</min>
+            <max>12.0</max> <!-- Maksymalny zasięg RPLIDAR A2M12 wynosi 12 metrów -->
+            </range>
+            <noise>
+            <type>gaussian</type>
+            <mean>0.0</mean>
+            <stddev>0.01</stddev>
+            </noise>
+        </ray>
+        <plugin name="gazebo_ros_range" filename="libgazebo_ros_range.so">
+            <topicName>/scan</topicName>
+            <frameName>lidar_link</frameName>
+        </plugin>
+        </sensor>
+    </gazebo>
 </robot>

File: src/pbl_description/urdf/salamanca.urdf.xacro (robot description, xacro)
@@ -2,4 +2,5 @@
 <robot name="salamanca" xmlns:xacro="http://www.ros.org/wiki/xacro">
     <xacro:include filename="common_properties.urdf.xacro" />
+    <xacro:include filename="mobile_base_gazebo.xacro"/>
     <xacro:include filename="mobile_base.urdf.xacro" />
 </robot>

Commit message: Gazebo fixed

File: src/pbl_description/urdf/mobile_base.urdf.xacro (robot description, xacro)
@@ -36,15 +36,16 @@
     <xacro:property name="battery_height" value="0.062" />
     <xacro:property name="battery_mass" value="1.974" />
-    <link name="base_footprint"></link>
+    <!-- <link name="base_footprint"></link> -->
     <link name="base_link">
         <visual>
             <geometry>
-                <mesh filename="package://pbl_description/stl/base_link.stl" scale="${scale_factor} ${scale_factor} ${scale_factor}" />
-            </geometry>
-            <origin xyz="0 0 0" rpy="0 0 0" />
-        </visual>
-        <collision>
-            <geometry>
-                <mesh filename="package://pbl_description/stl/base_link.stl" scale="${scale_factor} ${scale_factor} ${scale_factor}" />
+                <mesh filename="file://$(find pbl_description)/stl/base_link.stl" scale="${scale_factor} ${scale_factor} ${scale_factor}" />
+            </geometry>
+            <origin xyz="0 0 0" rpy="0 0 0" />
+        </visual>
+        <collision>
+            <geometry>
+                <!-- <mesh filename="file://$(find pbl_description)/stl/base_link.stl" scale="${scale_factor} ${scale_factor} ${scale_factor}" /> -->
+                <mesh filename="file://$(find pbl_description)/stl/base_link.stl" scale="${scale_factor} ${scale_factor} ${scale_factor}" />
             </geometry>
             <origin xyz="0 0 0" rpy="0 0 0" />
@@ -56,11 +57,11 @@
         <visual>
             <geometry>
-                <mesh filename="package://pbl_description/stl/castor_wheel.stl" scale="${scale_factor} ${scale_factor} ${scale_factor}" />
-            </geometry>
-            <origin xyz="0 0 0" rpy="0 0 0" />
-        </visual>
-        <collision>
-            <geometry>
-                <mesh filename="package://pbl_description/stl/castor_wheel.stl" scale="${scale_factor} ${scale_factor} ${scale_factor}" />
+                <mesh filename="file://$(find pbl_description)/stl/castor_wheel.stl" scale="${scale_factor} ${scale_factor} ${scale_factor}" />
+            </geometry>
+            <origin xyz="0 0 0" rpy="0 0 0" />
+        </visual>
+        <collision>
+            <geometry>
+                <mesh filename="file://$(find pbl_description)/stl/castor_wheel.stl" scale="${scale_factor} ${scale_factor} ${scale_factor}" />
             </geometry>
             <origin xyz="0 0 0" rpy="0 0 0" />
@@ -72,5 +73,5 @@
         <visual>
             <geometry>
-                <mesh filename="package://pbl_description/stl/realsense_camera.stl"
+                <mesh filename="file://$(find pbl_description)/stl/realsense_camera.stl"
                 scale="${scale_factor} ${scale_factor} ${scale_factor}" />
             </geometry>
@@ -79,5 +80,5 @@
         <collision>
             <geometry>
-                <mesh filename="package://pbl_description/stl/realsense_camera.stl"
+                <mesh filename="file://$(find pbl_description)/stl/realsense_camera.stl"
                 scale="${scale_factor} ${scale_factor} ${scale_factor}" />
             </geometry>
@@ -90,11 +91,11 @@
         <visual>
             <geometry>
-                <mesh filename="package://pbl_description/stl/jetson_nano.stl" scale="${scale_factor} ${scale_factor} ${scale_factor}" />
-            </geometry>
-            <origin xyz="0 0 0" rpy="0 0 0" />
-        </visual>
-        <collision>
-            <geometry>
-                <mesh filename="package://pbl_description/stl/jetson_nano.stl" scale="${scale_factor} ${scale_factor} ${scale_factor}" />
+                <mesh filename="file://$(find pbl_description)/stl/jetson_nano.stl" scale="${scale_factor} ${scale_factor} ${scale_factor}" />
+            </geometry>
+            <origin xyz="0 0 0" rpy="0 0 0" />
+        </visual>
+        <collision>
+            <geometry>
+                <mesh filename="file://$(find pbl_description)/stl/jetson_nano.stl" scale="${scale_factor} ${scale_factor} ${scale_factor}" />
             </geometry>
             <origin xyz="0 0 0" rpy="0 0 0" />
@@ -138,11 +139,11 @@
         <visual>
             <geometry>
-                <mesh filename="package://pbl_description/stl/rplidar_a2_mount.stl" scale="${scale_factor} ${scale_factor} ${scale_factor}" />
-            </geometry>
-            <origin xyz="0 0 0" rpy="0 0 0" />
-        </visual>
-        <collision>
-            <geometry>
-                <mesh filename="package://pbl_description/stl/rplidar_a2_mount.stl" scale="${scale_factor} ${scale_factor} ${scale_factor}" />
+                <mesh filename="file://$(find pbl_description)/stl/rplidar_a2_mount.stl" scale="${scale_factor} ${scale_factor} ${scale_factor}" />
+            </geometry>
+            <origin xyz="0 0 0" rpy="0 0 0" />
+        </visual>
+        <collision>
+            <geometry>
+                <mesh filename="file://$(find pbl_description)/stl/rplidar_a2_mount.stl" scale="${scale_factor} ${scale_factor} ${scale_factor}" />
             </geometry>
             <origin xyz="0 0 0" rpy="0 0 0" />
@@ -154,11 +155,11 @@
         <visual>
             <geometry>
-                <mesh filename="package://pbl_description/stl/tattu_battery.stl" scale="${scale_factor} ${scale_factor} ${scale_factor}" />
-            </geometry>
-            <origin xyz="0 0 0" rpy="0 0 0" />
-        </visual>
-        <collision>
-            <geometry>
-                <mesh filename="package://pbl_description/stl/tattu_battery.stl" scale="${scale_factor} ${scale_factor} ${scale_factor}" />
+                <mesh filename="file://$(find pbl_description)/stl/tattu_battery.stl" scale="${scale_factor} ${scale_factor} ${scale_factor}" />
+            </geometry>
+            <origin xyz="0 0 0" rpy="0 0 0" />
+        </visual>
+        <collision>
+            <geometry>
+                <mesh filename="file://$(find pbl_description)/stl/tattu_battery.stl" scale="${scale_factor} ${scale_factor} ${scale_factor}" />
             </geometry>
             <origin xyz="0 0 0" rpy="0 0 0" />
@@ -167,47 +168,53 @@
             xyz="0 0 0" rpy="0 0 0" />
     </link>
-    <joint name="base_joint" type="fixed">
-        <parent link="base_link" />
-        <child link="base_footprint" />
+    <!-- <joint name="base_joint" type="revolute">
+        <parent link="base_footprint" />
+        <child link="base_link" />
         <origin xyz="0 0 ${-odrive_radius+base_height}" rpy="0 0 0" />
-    </joint>
-    <joint name="castor_joint" type="fixed">
+        <limit lower="0.0" upper="0.0" effort="100.0" velocity="-1.0" />
+    </joint> -->
+    <joint name="castor_joint" type="revolute">
         <parent link="base_link" />
         <child link="castor_wheel" />
         <origin xyz="${-(2/7)*base_length + 0.01} 0 0" rpy="0 0 0" />
-    </joint>
-    <joint name="rplidar_mount_joint" type="fixed">
+        <limit lower="0.0" upper="0.0" effort="100.0" velocity="-1.0" />
+    </joint>
+    <joint name="rplidar_mount_joint" type="revolute">
         <parent link="base_link" />
         <child link="rplidar_a2_mount" />
         <origin xyz="0 0 0.095" rpy="0 0 0" />
-    </joint>
-    <joint name="realsense_joint" type="fixed">
+        <limit lower="0.0" upper="0.0" effort="100.0" velocity="-1.0" />
+    </joint>
+    <joint name="realsense_joint" type="revolute">
         <parent link="base_link" />
         <child link="realsense_camera" />
         <origin xyz="${(-base_length/2)+realsense_width} 0 ${base_height}" rpy="0 0 0" />
-    </joint>
-    <joint name="battery_joint" type="fixed">
+        <limit lower="0.0" upper="0.0" effort="100.0" velocity="-1.0" />
+    </joint>
+    <joint name="battery_joint" type="revolute">
         <parent link="base_link" />
         <child link="tattu_battery" />
         <origin xyz="-0.08 0 ${base_height}" rpy="0 0 0" />
-    </joint>
-    <joint name="jetson_joint" type="fixed">
+        <limit lower="0.0" upper="0.0" effort="100.0" velocity="-1.0" />
+    </joint>
+    <joint name="jetson_joint" type="revolute">
         <parent link="base_link" />
         <child link="jetson_nano" />
         <origin xyz="${base_length/3} 0 ${base_height}" rpy="0 0 0" />
-    </joint>
-    <joint name="left_wheel_joint" type="revolute">
+        <limit lower="0.0" upper="0.0" effort="100.0" velocity="-1.0" />
+    </joint>
+    <joint name="left_wheel_joint" type="continuous">
         <parent link="base_link" />
         <child link="odrive_bothwheel_l" />
-        <origin xyz="${odrive_radius + 0.04} ${(-base_width / 2) - (odrive_height/2)} ${base_height/2}" rpy="0 0 0" />
+        <origin xyz="${odrive_radius + 0.04} ${(-base_width / 2) - (odrive_height / 2)} ${base_height / 2}" rpy="0 0 0" />
         <axis xyz="0 1 0" />
-        <limit lower="-3.14159" upper="3.14159" effort="1" velocity="10" />
-    </joint>
-    <joint name="right_wheel_joint" type="revolute">
+        <dynamics damping="0.1" friction="0.0" />
+    </joint>
+    <joint name="right_wheel_joint" type="continuous">
         <parent link="base_link" />
         <child link="odrive_bothwheel_r" />
-        <origin xyz="${odrive_radius + 0.04} ${(base_width / 2) + (odrive_height/2)} ${base_height/2}" rpy="0 0 0" />
+        <origin xyz="${odrive_radius + 0.04} ${(base_width / 2) + (odrive_height / 2)} ${base_height / 2}" rpy="0 0 0" />
         <axis xyz="0 1 0" />
-        <limit lower="-3.14159" upper="3.14159" effort="1" velocity="10" />
+        <dynamics damping="0.1" friction="0.0" />
     </joint>
 </robot>

File: src/pbl_description/urdf/mobile_base_gazebo.xacro (robot description, xacro)
@@ -4,37 +4,41 @@
         <material>Gazebo/Yellow</material>
     </gazebo>
-    <gazebo reference="right_wheel_link">
+    <gazebo reference="castor_wheel">
         <material>Gazebo/Grey</material>
     </gazebo>
-    <gazebo reference="left_wheel_link">
+    <gazebo reference="realsense_camera">
         <material>Gazebo/Grey</material>
     </gazebo>
-    <gazebo reference="caster_wheel_link">
+    <gazebo reference="jetson_nano">
         <material>Gazebo/Grey</material>
-        <mu1 value="0.1" />
-        <mu2 value="0.1"/>
+    </gazebo>
+    <gazebo reference="odrive_bothwheel_r">
+        <material>Gazebo/Grey</material>
+    </gazebo>
+    <gazebo reference="odrive_bothwheel_l">
+        <material>Gazebo/Grey</material>
+    </gazebo>
+    <gazebo reference="rplidar_a2_mount">
+        <material>Gazebo/Grey</material>
+    </gazebo>
+    <gazebo reference="tattu_battery">
+        <material>Gazebo/Grey</material>
     </gazebo>
     <gazebo>
-        <plugin name="diff_drive_controller" filename="libgazebo_ros_diff_drive.so">
-            <!-- Update rate in Hz -->
-            <update_rate>50</update_rate>
-            <!-- wheels -->
-            <left_joint>left_wheel_joint</left_joint>
-            <right_joint>right_wheel_joint</right_joint>
-            <!-- kinematics -->
-            <wheel_separation>0.45</wheel_separation>
-            <wheel_diameter>0.2</wheel_diameter>
-            <!-- input -->
-            <command_topic>cmd_vel</command_topic>
-            <!-- output -->
-            <publish_odom>true</publish_odom>
-            <publish_odom_tf>true</publish_odom_tf>
-            <publish_wheel_tf>true</publish_wheel_tf>
-            <odometry_topic>odom</odometry_topic>
-            <odometry_frame>odom</odometry_frame>
-            <robot_base_frame>base_footprint</robot_base_frame>
-        </plugin>
-    </gazebo>
-    <!-- Plugin Gazebo for lidar -->
+            <plugin name="diff_drive_controller" filename="libgazebo_ros_diff_drive.so">
+                <update_rate>50</update_rate>
+                <left_joint>left_wheel_joint</left_joint>
+                <right_joint>right_wheel_joint</right_joint>
+                <wheel_separation>0.45</wheel_separation>
+                <wheel_diameter>0.2</wheel_diameter>
+                <command_topic>cmd_vel</command_topic>
+                <publish_odom>false</publish_odom>
+                <publish_odom_tf>false</publish_odom_tf>
+                <publish_wheel_tf>false</publish_wheel_tf>
+                <odometry_topic>odom</odometry_topic>
+                <odometry_frame>odom</odometry_frame>
+                <robot_base_frame>base_link</robot_base_frame>
+            </plugin>
+        </gazebo>
     <gazebo reference="rplidar_a2_mount">
         <sensor type="ray" name="lidar_sensor">
@@ -53,5 +57,5 @@
             <range>
             <min>0.15</min>
-            <max>12.0</max> <!-- Maksymalny zasięg RPLIDAR A2M12 wynosi 12 metrów -->
+            <max>12.0</max>
             </range>
             <noise>

Commit message: gl hf

File: src/pbl_description/urdf/mobile_base.urdf.xacro (robot description, xacro)
@@ -36,5 +36,5 @@
     <xacro:property name="battery_height" value="0.062" />
     <xacro:property name="battery_mass" value="1.974" />
-    <!-- <link name="base_footprint"></link> -->
+    <link name="base_footprint"></link>
     <link name="base_link">
         <visual>
@@ -168,10 +168,10 @@
             xyz="0 0 0" rpy="0 0 0" />
     </link>
-    <!-- <joint name="base_joint" type="revolute">
+    <joint name="base_joint" type="fixed">
         <parent link="base_footprint" />
         <child link="base_link" />
         <origin xyz="0 0 ${-odrive_radius+base_height}" rpy="0 0 0" />
-        <limit lower="0.0" upper="0.0" effort="100.0" velocity="-1.0" />
-    </joint> -->
+        <!-- <limit lower="0.0" upper="0.0" effort="100.0" velocity="-1.0" /> -->
+    </joint>
     <joint name="castor_joint" type="revolute">
         <parent link="base_link" />

File: src/pbl_description/urdf/mobile_base_gazebo.xacro (robot description, xacro)
@@ -19,5 +19,5 @@
         <pose>0 0 0 0 0 3.14</pose>
         <visualize>true</visualize>
-        <update_rate>10.0</update_rate>
+        <update_rate>10</update_rate>
         <!-- Camera Specifications -->
         <camera name="rpi_camera">
@@ -40,5 +40,5 @@
         <plugin name="raspberry_pi_hq_camera_plugin" filename="libgazebo_ros_camera.so">
         <alwaysOn>true</alwaysOn>
-        <updateRate>10.0</updateRate>
+        <updateRate>10</updateRate>
         <cameraName>salamanca/rpi_camera</cameraName>
         <imageTopicName>image_raw</imageTopicName>
@@ -60,10 +60,10 @@
         <pose>0 0 0 0 0 0</pose>
         <visualize>true</visualize>
-        <update_rate>10</update_rate>
+        <update_rate>10.0</update_rate>
         <ray>
             <scan>
             <horizontal>
-                <samples>360</samples>
-                <resolution>1</resolution>
+                <samples>360.0</samples>
+                <resolution>1.0</resolution>
                 <min_angle>-3.14159</min_angle>
                 <max_angle>3.14159</max_angle>
@@ -74,13 +74,11 @@
             <max>12.0</max> //for this lidar maximum distance is 12 m
             </range>
-            <noise>
-            <type>gaussian</type>
-            <mean>0.0</mean>
-            <stddev>0.01</stddev>
-            </noise>
         </ray>
-        <plugin name="gazebo_ros_range" filename="libgazebo_ros_range.so">
-            <topicName>/scan</topicName>
-            <frameName>lidar_link</frameName>
+        <plugin name="lidar" filename="libgazebo_ros_ray_sensor.so">
+            <output_type>sensor_msgs/LaserScan</output_type>
+            <ros>
+                <remapping>~/out:=scan</remapping>
+            </ros>
+            <frame_name>rplidar_a2_mount</frame_name>
         </plugin>
         </sensor>
@@ -94,5 +92,5 @@
     <gazebo>
             <plugin name="diff_drive_controller" filename="libgazebo_ros_diff_drive.so">
-                <update_rate>50</update_rate>
+                <update_rate>10</update_rate>
                 <left_joint>left_wheel_joint</left_joint>
                 <right_joint>right_wheel_joint</right_joint>
@@ -100,10 +98,10 @@
                 <wheel_diameter>0.2</wheel_diameter>
                 <command_topic>cmd_vel</command_topic>
-                <publish_odom>false</publish_odom>
-                <publish_odom_tf>false</publish_odom_tf>
+                <publish_odom>true</publish_odom>
+                <publish_odom_tf>true</publish_odom_tf>
                 <publish_wheel_tf>false</publish_wheel_tf>
                 <odometry_topic>odom</odometry_topic>
                 <odometry_frame>odom</odometry_frame>
-                <robot_base_frame>base_link</robot_base_frame>
+                <robot_base_frame>base_footprint</robot_base_frame>
             </plugin>
         </gazebo>
